File: Hardware/RedBot.sch (EAGLE design)
At the start: 66 parts, among them U1 ATMEGA328P, U2 TB6612FNG, U3 MIC5219 5V, U4 MIC5219 3.3V, U5 FT232RLSSOP, U6 7408SE, Y1 16MHz

Commit message: First pass at converting schematic
Parts:
- removed C5, C7: 0.1uF, SparkFun-Capacitors:0.1UF-25V(+80/-20%)(0603)
- removed D2: (no value), SparkFun-DiscreteSemi:B340A
- removed D3, D4, D5: GREEN, SparkFun-LED:LED-GREEN0603
- removed JP4: USB-B, SparkFun-Connectors:USB-MINIB-5PIN
- removed JP5: AVR_SPI_PRG_6PTH, SparkFun-Connectors:AVR_SPI_PRG_6PTH
- removed JP9: (no value), SparkFun-Connectors:M03X2SMT
- removed MOD1: XBEE-1B3, SparkFun-RF:XBEE-1B3
- removed R1, R12, R13: 10k, SparkFun-Resistors:10KOHM1/10W1%(0603)0603
- removed R2, R3, R4, R5, R6, R7: 1k, SparkFun-Resistors:1K-1%
- removed S3: DPDT, SparkFun-Electromechanical:SWITCH-DPDTAYZ0202
- removed S4: (no value), SparkFun-Electromechanical:TAC_SWITCHSMD
- removed SFE-LOGO1: LOGO-SFENEW, SparkFun-Aesthetics:LOGO-SFENEW
- removed U$21: FOUR_LAYER_WARNING, SparkFun-Aesthetics:FOUR_LAYER_WARNING
- removed U4: MIC5219 3.3V, SparkFun-PowerIC:V_REG_MIC52193.3V
- removed U5: FT232RLSSOP, SparkFun-DigitalIC:FT232RLSSOP
- removed U6: 7408SE, SparkFun-DigitalIC:7408SE
- removed Y1: 16MHz, SparkFun-FreqCtrl:RESONATOR16MHZ
- added LAUNCHPAD: BOOSTERPACK, zlalanne:BOOSTERPACK
Connections:
- removed net AREF: U1.AREF
- removed net FT232_RXI: R3.1, U5.RXD
- removed net FT232_TXO: R2.1, U5.TXD
- removed net FTDI_DTR: R13.1, U5.DTR, U6.A
- removed net N$1: R4.2, S3.2
- removed net N$23: U1.PB7(XTAL2/TOSC2), Y1.3
- removed net N$24: U1.PB6(XTAL1/TOSC1), Y1.1
- removed net N$26: JP4.D-, U5.USBDM
- removed net N$27: JP4.D+, U5.USBDP
- removed net N$3: D5.C, R6.1
- removed net N$4: D3.C, R5.1
- removed net N$5: C7.2, U6.Y
- removed net N$6: JP4.MTN1, JP4.MTN2, JP4.MTN3, JP4.MTN4
- removed net N$7: D4.A, R7.1
- removed net RESET: C7.1, JP5.5, R1.2, S4.3, U1.PC6(/RESET)
- removed net RXI: R2.2, S3.4, U1.PD0(RXD)
- removed net RXLED: R5.2, U5.RXLED
- removed net SENSOR_0/SW_TXO: JP10.1, S3.3, U1.PC0(ADC0)
- removed net SENSOR_1/SW_RXI: JP10.2, S3.6, U1.PC1(ADC1)
- removed net SERVO_3: JP9.1, U1.PB2(SS/OC1B)
- removed net TXLED: R6.2, U5.TXLED
- removed net TXO: R3.2, S3.1, U1.PD1(TXD)
- removed net V_USB: C5.1, D2.A, D3.A, D5.A, JP4.VBUS, U5.VCC, U5.VCCIO
- removed net XBEE_DIO3: MOD1.DIO3, R12.1, U6.B
- removed net XBEE_RXI: MOD1.DIN, R4.1
- removed net XBEE_TXO: MOD1.DOUT, S3.5
- new net PWM_L: LAUNCHPAD.PWM_D1/GPIO_I_D1
- new net PWM_R: LAUNCHPAD.PWM_D2/GPIO_I_D2
- new net SENSOR_0: JP10.1, LAUNCHPAD.AIN_C1
- new net SENSOR_1: JP10.2, LAUNCHPAD.AIN_C2
- net 3.3V: now also JP10.3, JP10.4, JP11.3, JP11.4, JP12.3, JP12.4, JP13.3, JP13.4, JP7.1, JP7.3, JP7.5, JP7.7, JP7.9, LAUNCHPAD.3V3; no longer MOD1.VDD, U4.OUT
- net 5V: now also LAUNCHPAD.5V; no longer JP10.3, JP10.4, JP11.3, JP11.4, JP12.3, JP12.4, JP13.3, JP13.4, JP5.2, JP7.1, JP7.3, JP7.5, JP7.7, JP7.9, R1.1, R12.2, R13.2, U1.AVCC, U1.VCC@1, U1.VCC@2, U4.EN, U4.IN, U6.VCC
- net GND: now also LAUNCHPAD.GND, LAUNCHPAD.GND2; no longer C5.2, D4.C, JP4.GND, JP5.6, JP9.5, JP9.6, MOD1.GND, S4.1, U1.AGND, U1.GND@1, U1.GND@2, U4.GND, U5.AGND, U5.GND18, U5.GND21, U5.GND7, U5.TEST, U6.GND, Y1.2
- net L_CTRL_1: now also LAUNCHPAD.GPIO_I_D7; no longer U1.PD2(INT0)
- net L_CTRL_2: now also LAUNCHPAD.GPIO_I_D8
- net MISO: no longer JP5.1
- net PWML: no longer U1.PD5(T1)
- net PWMR: no longer U1.PD6(AIN0)
- net R_CTRL_1: now also LAUNCHPAD.GPIO_I_D9; no longer U1.PD7(AIN1)
- net R_CTRL_2: now also LAUNCHPAD.GPIO_I_D10; no longer U1.PB0(ICP)
- net SCK: no longer JP5.3, R7.2
- net SENSOR_2: now also LAUNCHPAD.AIN_C3; no longer U1.PC2(ADC2)
- net SENSOR_3: now also LAUNCHPAD.AIN_C4; no longer U1.PC3(ADC3)
- net SENSOR_4: now also LAUNCHPAD.AIN_C5/I2S_WS; no longer U1.PC4(ADC4/SDA)
- net SENSOR_5: now also LAUNCHPAD.AIN_C6/I2S_SCLK; no longer U1.PC5(ADC5/SCL)
- net SENSOR_6: now also LAUNCHPAD.AIN_A1; no longer U1.ADC6
- net SENSOR_7: now also LAUNCHPAD.AIN_A2; no longer U1.ADC7
- net SERVO_1: now also LAUNCHPAD.PWM_D3/GPIO_I_D3
- net SERVO_2: now also LAUNCHPAD.PWM_D4/GPIO_I_D4
- net SERVO_4/MOSI: no longer JP5.4, JP9.2
- net V_GATED: no longer JP9.3, JP9.4
- net V_IN: no longer D2.C
Other:
- moved on the sheet: JP10, JP11, JP12, JP13, JP8
